File: hydra open souce project/Hydra OSP.brd (EAGLE design)
At the start: 78.4 x 55.9 mm, 9 parts, among them X1 1-227161-2, X2 1-227161-2

Commit message: DRC eurocircuits
Parts:
- added SV3: (no value), con-lstb:MA05-2
- SV1: value 1 -> (none); device con-lstb:MA10-2 -> con-lstb:MA08-2
- moved SV1 5.94 mm to (61.0, 50.0)
Connections:
- net 1WIRE: now also SV1.2, SV1.4; no longer SV1.18, SV1.20
- net GND: now also SV3.1, SV3.3, SV3.5, SV3.7, SV3.9; no longer SV1.3, SV1.4
- net RX_I2C: now also SV1.3; no longer SV1.19
- net TX_I2C: now also SV1.1; no longer SV1.17
- net VCC: now also SV3.10, SV3.2, SV3.4, SV3.6, SV3.8; no longer SV1.1, SV1.2
Routing:
- net VCC: track 83.2 -> 112.1 mm
- net TX_I2C: track 57.6 -> 84.2 mm
- net RX_I2C: track 73.6 -> 77.9 mm
- net 1WIRE: track 52.7 -> 54.3 mm
Other:
- board text added: "Hydra Open Source Project"
- board text removed: "hHydra Open Source Project"
