File: hydra open souce project/Hydra OSP.sch (EAGLE design)
At the start: 9 parts, among them X1 1-227161-2, X2 1-227161-2

Commit message: DRC eurocircuits
Parts:
- added SV3: (no value), con-lstb:MA05-2
- SV1: value 1 -> (none); device con-lstb:MA10-2 -> con-lstb:MA08-2
Connections:
- net 1WIRE: now also SV1.2, SV1.4; no longer SV1.18, SV1.20
- net GND: now also SV3.1, SV3.3, SV3.5, SV3.7, SV3.9; no longer SV1.3, SV1.4
- net RX_I2C: now also SV1.3; no longer SV1.19
- net TX_I2C: now also SV1.1; no longer SV1.17
- net VCC: now also SV3.10, SV3.2, SV3.4, SV3.6, SV3.8; no longer SV1.1, SV1.2
Other:
- note added: "1Wire devices: 8 I2C devices: 4"
- note added: "POWER 3V3"
- note added: "SENSORS"
- note removed: "Hydra Open Source Project"
